File: Schmatics/KiCAD Schematics/6502 Computer.kicad_sch (KiCad schematic)
At the start: 47 parts, among them J10 Conn_02x01, J11 RCJ-017, J12 Conn_02x03_Odd_Even, J2 Conn_02x20_Odd_Even, J3 Conn_01x04_Male, J4 Conn_02x03_Odd_Even, J5 Conn_02x08_Odd_Even, J6 Conn_01x06_Male, J7 Conn_02x03_Odd_Even, J8 Barrel_Jack, J9 Conn_01x11_Male, P1 Mini-DIN_6pins, SW1 RESET, U1 WD65C02, U2 28C256, U3 WC1602A, U4 74HC00, U5 WD65C22, U6 CY62256-70PC, U7 6551, U8 74HC166, X1 ACO-1.8432MHz, Y1 11.0582 MHz, Y2 16 MHz

Commit message: Scripts and Stuff
Parts:
- removed C15: 10uF, Capacitor_SMD:CP_Elec_4x3.9, symbol 6502 Computer-rescue:CP1-Device
- added C13, C15: 10uf, Capacitor_THT:C_Radial_D5.0mm_H11.0mm_P2.00mm, symbol Device:C
- added J13: Conn_02x01, Connector_PinHeader_2.54mm:PinHeader_2x01_P2.54mm_Vertical, symbol Connector_Generic:Conn_02x01
- added U9: LM7805_TO220, Package_TO_SOT_THT:TO-220-3_Vertical, symbol Regulator_Linear:LM7805_TO220
Connections:
- net +5V: now also C15.1, U9.3 (VO); no longer J8.1, R6.1
- net GND: now also R6.1, C13.2, C15.2, U9.2 (GND)
- net at J2.8 (Pin_8), U1.37 (PHI2), U4.9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: now also J13.1 (Pin_1); no longer X1.8 (OUT)
- net at J5.11 (Pin_11), U5.7 (PA5): now also J12.4 (Pin_4); no longer J12.2 (Pin_2)
- net at J5.15 (Pin_15), U5.9 (PA7): now also J12.3 (Pin_3); no longer J12.1 (Pin_1)
- net at U3.4 (RS): now also J12.2 (Pin_2); no longer J12.4 (Pin_4)
- net at U3.6 (E): now also J12.1 (Pin_1); no longer J12.3 (Pin_3)
- new net: J13.2 (Pin_2), X1.8 (OUT)
- new net: C13.1, J8.1, U9.1 (VI)
Other:
- moved on the sheet: J8

Commit message: MAJOR push with big basic improvements
Parts:
- removed J10: Conn_02x01, Connector_PinHeader_2.54mm:PinHeader_2x01_P2.54mm_Vertical, symbol Connector_Generic:Conn_02x01
- removed J6: Conn_01x06_Male, Connector_PinHeader_2.54mm:PinHeader_1x06_P2.54mm_Horizontal, symbol 6502 Computer-rescue:Conn_01x06_Male-Connector
- added C16, C17, C18, C19: 1uf, Capacitor_THT:C_Disc_D4.3mm_W1.9mm_P5.00mm, symbol Device:C
- added J1: DE9_Pins, Connector_Dsub:DSUB-9_Socket_Horizontal_P2.77x2.54mm_EdgePinOffset9.40mm, symbol Connector:DE9_Pins
- added J10: Conn_01x01, Connector_PinHeader_2.00mm:PinHeader_1x01_P2.00mm_Vertical, symbol Connector_Generic:Conn_01x01
- added J14, J15, J16: Conn_02x01, Connector_PinHeader_2.54mm:PinHeader_2x01_P2.54mm_Vertical, symbol Connector_Generic:Conn_02x01
- added J6: Conn_01x03, Connector_PinHeader_2.00mm:PinHeader_1x03_P2.00mm_Vertical, symbol Connector_Generic:Conn_01x03
- added R7, R8, R9: 10k, Resistor_THT:R_Axial_DIN0204_L3.6mm_D1.6mm_P7.62mm_Horizontal, symbol Device:R
- added U10: MAX232, Package_DIP:DIP-16_W7.62mm, symbol Interface_UART:MAX232
- SW1: footprint Button_Switch_THT:SW_PUSH_6mm_H5mm -> Button_Switch_THT:SW_PUSH_1P1T_6x3.5mm_H4.3_APEM_MJTP1243
Connections:
- net +5V: now also J14.2 (Pin_2), J15.2 (Pin_2), R7.2, R8.1, R9.1, U10.16 (VCC); no longer J7.1 (Pin_1), J7.3 (Pin_3), J7.5 (Pin_5), UA1.1 (~{RESET}/PC6), UB1.1 (~{RESET}/PC6)
- net GND: now also C17.1, C19.2, J1.5, U10.15 (GND)
- net at J13.1 (Pin_1), J2.8 (Pin_8), U1.37 (PHI2)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: now also J16.2 (Pin_2); no longer U7.6 (XTLI)
- net at J2.7 (Pin_7), J7.4 (Pin_4), U1.4 (~{IRQ}): now also J6.2 (Pin_2); no longer U5.21 (~{IRQ})
- net at C5.1, J2.2 (Pin_2), R1.2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: now also UA1.1 (~{RESET}/PC6), UB1.1 (~{RESET}/PC6)
- net at UA1.26 (PC3): now also U7.8 (~{RTS}), U10.10 (T2IN)
- net at U7.26 (~{IRQ}): now also J14.1 (Pin_1), J6.1 (Pin_1)
- net at U7.7 (XLT0): now also J10.1 (Pin_1)
- net at J4.5 (Pin_5): now also U10.11 (T1IN)
- net at J4.6 (Pin_6): now also U10.12 (R1OUT)
- new net: J15.1 (Pin_1), J6.3 (Pin_3), U5.21 (~{IRQ})
- new net: J16.1 (Pin_1), U7.6 (XTLI)
- new net: J7.1 (Pin_1), R7.1
- new net: J7.3 (Pin_3), R9.2
- new net: J7.5 (Pin_5), R8.2
- new net: C19.1, U10.6 (VS-)
- new net: J1.2, U10.13 (R1IN)
- new net: J1.3, U10.14 (T1OUT)
- new net: J1.7, U10.7 (T2OUT)
- new net: C16.1, U10.1 (C1+)
- new net: C17.2, U10.2 (VS+)
- new net: C16.2, U10.3 (C1-)
- new net: C18.1, U10.4 (C2+)
- new net: C18.2, U10.5 (C2-)
- no-connect marks 16 -> 17

Commit message: Schumatic Sound Chip
Parts:
- removed C13, C15: 10uf, Capacitor_THT:C_Radial_D5.0mm_H11.0mm_P2.00mm, symbol Device:C
- removed J10: Conn_01x01, Connector_PinHeader_2.00mm:PinHeader_1x01_P2.00mm_Vertical, symbol Connector_Generic:Conn_01x01
- removed J13, J16: Conn_02x01, Connector_PinHeader_2.54mm:PinHeader_2x01_P2.54mm_Vertical, symbol Connector_Generic:Conn_02x01
- removed U9: LM7805_TO220, Package_TO_SOT_THT:TO-220-3_Vertical, symbol Regulator_Linear:LM7805_TO220
- added C13: 10uf, Capacitor_THT:CP_Radial_D4.0mm_P2.00mm, symbol Device:C_Polarized
- added C20: 0.05uF, Capacitor_THT:C_Radial_D5.0mm_H11.0mm_P2.00mm, symbol Device:C
- added C21: 20uF, Capacitor_THT:C_Radial_D5.0mm_H11.0mm_P2.00mm, symbol Device:C
- added J17: RCJ-017, Connector_RCA:CUI_RCJ-017, symbol RCA:RCJ-017
- added LS1: Speaker, Connector_PinHeader_2.00mm:PinHeader_1x02_P2.00mm_Vertical, symbol Device:Speaker
- added R10: 10 Ohm, Resistor_THT:R_Axial_DIN0204_L3.6mm_D1.6mm_P7.62mm_Horizontal, symbol Device:R
- added RV2: R_POT_TRIM_US, Potentiometer_THT:Potentiometer_Bourns_3386C_Horizontal, symbol 6502 Computer-rescue:R_POT_TRIM_US-Device
- added SN76489-AN1: ~, Package_DIP:DIP-16_W7.62mm, symbol SN:SN76489-AN
- added U11: LM386, Package_DIP:DIP-8_W7.62mm_Socket, symbol Amplifier_Audio:LM386
- added U12, U13: 74HC00, Package_DIP:DIP-14_W7.62mm_Socket_LongPads, symbol 74xx:74HC00
- added X2: 4MHz, Oscillator:Oscillator_DIP-14, symbol 6502 Computer-rescue:ACO-xxxMHz-Oscillator
Connections:
- net +5V: now also J8.1, C13.1, SN76489-AN1.16 (VCC), U11.6 (V+), U12.14 (VCC), U13.14 (VCC), X2.14 (Vcc)
- net GND: now also C13.2, J17.1A, J17.1B, J17.1C, LS1.2, R10.1, RV2.3, SN76489-AN1.8 (GND), U11.2 (-), U11.4 (GND), U12.7 (GND), U13.12, U13.13, U13.7 (GND), X2.7 (GND)
- net at J2.3 (Pin_3), J7.2 (Pin_2), U1.2 (RDY): now also SN76489-AN1.4 (RDY)
- net at J2.38 (Pin_38), U1.22 (A12), U2.2 (A12)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: now also U12.13
- net at J2.36 (Pin_36), U1.23 (A13), U2.26 (A13)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: now also U12.1, U12.10; no longer U5.24 (CS1)
- net at J2.34 (Pin_34), U1.24 (A14), U2.1 (A14)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: now also U12.9
- net at J2.30 (Pin_30), U1.26 (D7), U2.19 (D7)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: now also SN76489-AN1.10 (D7)
- net at J2.28 (Pin_28), U1.27 (D6), U2.18 (D6)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: now also SN76489-AN1.11 (D6)
- net at J2.26 (Pin_26), U1.28 (D5), U2.17 (D5)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: now also SN76489-AN1.12 (D5)
- net at J2.24 (Pin_24), U1.29 (D4), U2.16 (D4)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: now also SN76489-AN1.13 (D4)
- net at J2.22 (Pin_22), U1.30 (D3), U2.15 (D3)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: now also SN76489-AN1.15 (D3)
- net at J2.20 (Pin_20), U1.31 (D2), U2.13 (D2)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: now also SN76489-AN1.1 (D2)
- net at J2.18 (Pin_18), U1.32 (D1), U2.12 (D1)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: now also SN76489-AN1.2 (D1)
- net at J2.16 (Pin_16), U1.33 (D0), U2.11 (D0)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: now also SN76489-AN1.3 (D0)
- net at J2.14 (Pin_14), U1.34 (R/~{W}), U5.22 (R/~{W})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: now also SN76489-AN1.5 (WE_)
- net at J2.8 (Pin_8), U1.37 (PHI2), U4.9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: now also U7.6 (XTLI), X1.8 (OUT)
- net at U2.20 (~{CS}), U4.10, U4.11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: now also U12.12
- new net: U12.6, U5.24 (CS1)
- new net: U12.11, U13.4, U13.5
- new net: U13.10, U13.6
- new net: SN76489-AN1.6 (CE_), U12.2, U13.8
- new net: U13.3, U13.9
- new net: SN76489-AN1.14 (CLK), X2.8 (OUT)
- new net: RV2.1, SN76489-AN1.7 (A_Out)
- new net: U12.8, U13.1, U13.2
- new net: U12.3, U12.4, U12.5
- new net: RV2.2, U11.3 (+)
- new net: C20.1, C21.1, U11.5
- new net: C21.2, J17.1 (V_In), LS1.1
- new net: C20.2, R10.2
- no-connect marks 17 -> 22
